Commit message: update urdf

File: hexapod_description/urdf/ancabot.xacro (robot description, xacro)
@@ -74,12 +74,61 @@
             </inertial>
         </link>
+        <!-- coxa -->
+        <joint name="coxa_joint_${side}${position}" type="revolute">
+            <origin xyz="0.0 0.0 ${-body_height}" rpy="0.0 0.0 ${angle}"/>
+            <parent link="leg_center_${side}${position}"/>
+            <child link="coxa_${side}${position}"/>
+            <axis xyz="0.0 0.0 1.0"/>
+            <limit lower="${joint_lower_limit}" upper="${joint_upper_limit}" effort="${joint_effort}" velocity="${joint_velocity}"/>
+        </joint>
+        <transmission name="coxa_transmission_${side}${position}">
+            <type>transmission_interface/SimpleTransmission</type>
+            <joint name="coxa_joint_${side}${position}">
+                <hardwareInterface>EffortJointInterface</hardwareInterface>
+            </joint>
+            <actuator name="coxa_motor_${side}${position}">
+                <hardwareInterface>EffortJointInterface</hardwareInterface>
+                <mechanicalReduction>1</mechanicalReduction>
+            </actuator>
+        </transmission>
+        <link name="coxa_${side}${position}">
+            <visual>
+                <origin xyz="0.035 0.02 0.02" rpy="${-pi/2} 0.0 ${pi}"/>
+                <geometry>
+                    <mesh filename="package://hexapod_description/meshes/coxa.stl" scale="0.001 0.001 0.001"/>
+                </geometry>
+                <material name="">
+                    <color rgba="0.7 0.7 0.7 1"/>
+                </material>
+            </visual>
+            <collision>
+                <origin xyz="0.015 0.0 0.0" rpy="0.0 0.0 0.0" />
+                <geometry>
+                    <box size="0.05 0.04 0.035"/>
+                </geometry>
+                <material name="">
+                    <color rgba="0.7 0.7 0.7 1" />
+                </material>
+            </collision>
+            <inertial>
+                <origin xyz="0.0 0.0 0.0" rpy="0.0 0.0 0.0" />
+                <mass value="0.00001"/>
+                <inertia
+                    ixx="1.0" ixy="0.0"  ixz="0.0"
+                    iyy="1.0" iyz="0.0"
+                    izz="1.0" />
+            </inertial>
+        </link>
+        <gazebo reference="coxa_${side}${position}">
+            <material>Gazebo/DarkGrey</material>
+        </gazebo>
     </xacro:macro>
     <!-- Build robot model -->
     <!-- Build robot model -->
-    <xacro:leg side="R"     position="R"    x="-0.05825"   y="0.0935"     angle="-${pi*3/4}"     axis="1"/>
-    <xacro:leg side="R"     position="M"    x="-0.06225"   y="0.0250"     angle="-${pi/2}"       axis="1"/>
-    <xacro:leg side="R"     position="F"    x="-0.05825"   y="-0.0435"    angle="-${pi/4}"       axis="1"/>
-    <xacro:leg side="L"     position="R"    x="0.05825"    y="0.0935"     angle="${pi*3/4}"      axis="-1"/>
-    <xacro:leg side="L"     position="M"    x="0.06225"    y="0.0250"     angle="${pi/2}"        axis="-1"/>
-    <xacro:leg side="L"     position="F"    x="0.05825"    y="-0.0435"    angle="${pi/4}"        axis="-1"/>
+    <xacro:leg side="R"     position="R"    x="-0.05825"   y="0.0935"     angle="${pi*3/4}"     axis="1"/>
+    <xacro:leg side="R"     position="M"    x="-0.06225"   y="0.0250"     angle="${-pi}"      axis="1"/>
+    <xacro:leg side="R"     position="F"    x="-0.05825"   y="-0.0435"    angle="${-pi*3/4}"    axis="1"/>
+    <xacro:leg side="L"     position="R"    x="0.05825"    y="0.0935"     angle="${pi/4}"       axis="-1"/>
+    <xacro:leg side="L"     position="M"    x="0.06225"    y="0.0250"     angle="${-pi*2}"       axis="-1"/>
+    <xacro:leg side="L"     position="F"    x="0.05825"    y="-0.0435"    angle="${-pi/4}"      axis="-1"/>
 </robot>

Commit message: update

File: hexapod_description/urdf/ancabot.xacro (robot description, xacro)
@@ -5,7 +5,6 @@
     <xacro:property     name="body_width"       value="0.1525"/>
     <xacro:property     name="body_height"      value="0.0405"/>
-    <xacro:property     name="coxa_length"      value="0.0"/>
-    <xacro:property     name="femur_length"     value="0.0"/>
-    <xacro:property     name="tibia_length"     value="0.0"/>
+    <xacro:property     name="coxa_length"      value="0.02245"/>
+    <xacro:property     name="femur_length"     value="0.042"/>
     <xacro:property     name="ground_offset"    value="0.064" />
     <gazebo>
@@ -17,5 +16,5 @@
     <link name="body_link">
         <visual>
-            <origin xyz="${body_width/2} ${-body_length/2} ${body_height/2}" rpy="0.0 ${pi} 0.0"/>
+            <origin xyz="-${body_width/2} ${body_length/2 + 0.05} ${body_height/2}" rpy="0.0 ${pi} ${pi}"/>
             <geometry>
                 <mesh filename="package://hexapod_description/meshes/body.stl" scale="0.001 0.001 0.001"/>
@@ -26,7 +25,7 @@
         </visual>
         <collision>
-            <origin xyz="0.0 0.0 0.0" rpy="0.0 0.0 0.0"/>
+            <origin xyz="-${body_width/2} ${body_length/2 + 0.05} ${body_height/2}" rpy="0.0 ${pi} ${pi}"/>
             <geometry>
-                <box size="${body_width} ${body_length} ${body_height}"/>
+                <mesh filename="package://hexapod_description/meshes/body.stl" scale="0.001 0.001 0.001"/>
             </geometry>
             <material name="">
@@ -103,10 +102,10 @@
             </visual>
             <collision>
-                <origin xyz="0.015 0.0 0.0" rpy="0.0 0.0 0.0" />
-                <geometry>
-                    <box size="0.05 0.04 0.035"/>
-                </geometry>
-                <material name="">
-                    <color rgba="0.7 0.7 0.7 1" />
+                <origin xyz="0.035 0.02 0.02" rpy="${-pi/2} 0.0 ${pi}"/>
+                <geometry>
+                    <mesh filename="package://hexapod_description/meshes/coxa.stl" scale="0.001 0.001 0.001"/>
+                </geometry>
+                <material name="">
+                    <color rgba="0.7 0.7 0.7 1"/>
                 </material>
             </collision>
@@ -121,4 +120,102 @@
         </link>
         <gazebo reference="coxa_${side}${position}">
+            <material>Gazebo/DarkGrey</material>
+        </gazebo>
+        <!-- femur -->
+        <joint name="femur_joint_${side}${position}" type="revolute">
+            <origin xyz="${coxa_length} 0.0 0.0" rpy="${pi/2} ${pi/2} 0.0"/>
+            <parent link="coxa_${side}${position}"/>
+            <child link="femur_${side}${position}"/>
+            <axis xyz="0.0 0.0 ${-axis}"/>
+            <limit lower="${joint_lower_limit}" upper="${joint_upper_limit}" effort="${joint_effort}" velocity="${joint_velocity}"/>
+        </joint>
+        <transmission name="femur_transmission_${side}${position}">
+            <type>transmission_interface/SimpleTransmission</type>
+            <joint name="femur_joint_${side}${position}">
+                <hardwareInterface>EffortJointInterface</hardwareInterface>
+            </joint>
+            <actuator name="femur_motor_${side}${position}">
+                <hardwareInterface>EffortJointInterface</hardwareInterface>
+                <mechanicalReduction>1</mechanicalReduction>
+            </actuator>
+        </transmission>
+        <link name="femur_${side}${position}">
+            <visual>
+                <origin xyz="-0.03575 -0.0125 0.0285" rpy="0.0 ${pi} ${3*pi/2}"/>
+                <geometry>
+                    <mesh filename="package://hexapod_description/meshes/femur.stl" scale="0.001 0.001 0.001"/>
+                </geometry>
+                <material name="">
+                    <color rgba="0.7 0.7 0.7 1"/>
+                </material>
+            </visual>
+            <collision>
+                <origin xyz="-0.03575 -0.0125 0.0285" rpy="0.0 ${pi} ${3*pi/2}"/>
+                <geometry>
+                    <mesh filename="package://hexapod_description/meshes/femur.stl" scale="0.001 0.001 0.001"/>
+                </geometry>
+                <material name="">
+                    <color rgba="0.7 0.7 0.7 1"/>
+                </material>
+            </collision>
+            <inertial>
+                <origin xyz="0.0 0.0 0.0" rpy="0.0 0.0 0.0" />
+                <mass value="0.00001"/>
+                <inertia
+                    ixx="1.0" ixy="0.0"  ixz="0.0"
+                    iyy="1.0" iyz="0.0"
+                    izz="1.0" />
+            </inertial>
+        </link>
+        <gazebo reference="femur_${side}${position}">
+            <material>Gazebo/DarkGrey</material>
+        </gazebo>
+        <!-- tibia -->
+        <joint name="tibia_joint_${side}${position}" type="revolute">
+            <origin xyz="0.0 ${femur_length} 0.0" rpy="0.0 0.0 0.0"/>
+            <parent link="femur_${side}${position}"/>
+            <child link="tibia_${side}${position}"/>
+            <axis xyz="0.0 0.0 ${-axis}"/>
+            <limit lower="${joint_lower_limit}" upper="${joint_upper_limit}" effort="${joint_effort}" velocity="${joint_velocity}"/>
+        </joint>
+        <transmission name="tibia_transmission_${side}${position}">
+            <type>transmission_interface/SimpleTransmission</type>
+            <joint name="tibia_joint_${side}${position}">
+                <hardwareInterface>EffortJointInterface</hardwareInterface>
+            </joint>
+            <actuator name="tibia_motor_${side}${position}">
+                <hardwareInterface>EffortJointInterface</hardwareInterface>
+                <mechanicalReduction>1</mechanicalReduction>
+            </actuator>
+        </transmission>
+        <link name="tibia_${side}${position}">
+            <visual>
+                <origin xyz="0.02285 -0.01325 -0.0205" rpy="0.0 0.0 ${pi/2}"/>
+                <geometry>
+                    <mesh filename="package://hexapod_description/meshes/tibia.stl" scale="0.001 0.001 0.001"/>
+                </geometry>
+                <material name="">
+                    <color rgba="0.7 0.7 0.7 1"/>
+                </material>
+            </visual>
+            <collision>
+                <origin xyz="0.02285 -0.01325 -0.0205" rpy="0.0 0.0 ${pi/2}"/>
+                <geometry>
+                    <mesh filename="package://hexapod_description/meshes/tibia.stl" scale="0.001 0.001 0.001"/>
+                </geometry>
+                <material name="">
+                    <color rgba="0.7 0.7 0.7 1"/>
+                </material>
+            </collision>
+            <inertial>
+                <origin xyz="0.0 0.0 0.0" rpy="0.0 0.0 0.0" />
+                <mass value="0.00001"/>
+                <inertia
+                    ixx="1.0" ixy="0.0"  ixz="0.0"
+                    iyy="1.0" iyz="0.0"
+                    izz="1.0" />
+            </inertial>
+        </link>
+        <gazebo reference="tibia_${side}${position}">
             <material>Gazebo/DarkGrey</material>
         </gazebo>
@@ -126,8 +223,8 @@
     <!-- Build robot model -->
     <xacro:leg side="R"     position="R"    x="-0.05825"   y="0.0935"     angle="${pi*3/4}"     axis="1"/>
-    <xacro:leg side="R"     position="M"    x="-0.06225"   y="0.0250"     angle="${-pi}"      axis="1"/>
+    <xacro:leg side="R"     position="M"    x="-0.06225"   y="0.0250"     angle="${-pi}"        axis="1"/>
     <xacro:leg side="R"     position="F"    x="-0.05825"   y="-0.0435"    angle="${-pi*3/4}"    axis="1"/>
     <xacro:leg side="L"     position="R"    x="0.05825"    y="0.0935"     angle="${pi/4}"       axis="-1"/>
-    <xacro:leg side="L"     position="M"    x="0.06225"    y="0.0250"     angle="${-pi*2}"       axis="-1"/>
+    <xacro:leg side="L"     position="M"    x="0.06225"    y="0.0250"     angle="${-pi*2}"      axis="-1"/>
     <xacro:leg side="L"     position="F"    x="0.05825"    y="-0.0435"    angle="${-pi/4}"      axis="-1"/>
 </robot>

Commit message: add gazebo configuration file

File: hexapod_description/urdf/ancabot.xacro (robot description, xacro)
@@ -7,5 +7,5 @@
     <xacro:property     name="coxa_length"      value="0.02245"/>
     <xacro:property     name="femur_length"     value="0.042"/>
-    <xacro:property     name="ground_offset"    value="0.064" />
+    <xacro:property     name="ground_offset"    value="0.10" />
     <gazebo>
         <plugin name="gazebo_ros_control" filename="libgazebo_ros_control.so">

Commit message: ...

File: hexapod_description/urdf/ancabot.xacro (robot description, xacro)
@@ -7,5 +7,6 @@
     <xacro:property     name="coxa_length"      value="0.02245"/>
     <xacro:property     name="femur_length"     value="0.042"/>
-    <xacro:property     name="ground_offset"    value="0.10" />
+    <xacro:property     name="tibia_length"     value="0.0665"/>
+    <xacro:property     name="ground_offset"    value="0.065" />
     <gazebo>
         <plugin name="gazebo_ros_control" filename="libgazebo_ros_control.so">
@@ -51,8 +52,56 @@
     </joint>
     <!-- Joint properties -->
-    <xacro:property name="joint_lower_limit" value="-${3.14}"/>
-    <xacro:property name="joint_upper_limit" value="${3.14}"/>
+    <xacro:property name="joint_lower_limit" value="-${2.0}"/>
+    <xacro:property name="joint_upper_limit" value="${2.0}"/>
     <xacro:property name="joint_effort" value="6.0"/>
     <xacro:property name="joint_velocity" value="0.524"/>
+    <!-- Head properties -->
+    <joint name="pan_joint" type="revolute">
+        <parent link="body_link"/>
+        <child link="pan_link"/>
+        <origin xyz="0.0 0.1585 -0.0025" rpy="0.0 ${pi/2} 0.0"/>
+        <axis xyz="0.0 0.0 -1.0"/>
+        <limit lower="${joint_lower_limit}" upper="${joint_upper_limit}" effort="${joint_effort}" velocity="${joint_velocity}"/>
+    </joint>
+    <transmission name="pan_transmission">
+        <type>transmission_interface/SimpleTransmission</type>
+        <joint name="pan_joint">
+            <hardwareInterface>hardware_interface/EffortJointInterface</hardwareInterface>
+        </joint>
+        <actuator name="pan_motor">
+            <hardwareInterface>hardware_interface/EffortJointInterface</hardwareInterface>                <mechanicalReduction>1</mechanicalReduction>
+        </actuator>
+    </transmission>
+    <link name="pan_link">
+        <visual>
+            <origin xyz="0.1175 -0.0415 0.02785" rpy="0.0 ${pi/2} ${pi/2}"/>
+            <geometry>
+                <mesh filename="package://hexapod_description/meshes/gripper_hand.stl" scale="0.001 0.001 0.001"/>
+            </geometry>
+            <material name="">
+                <color rgba="0.7 0.7 0.7 1"/>
+            </material>
+        </visual>
+        <collision>
+            <origin xyz="0.1175 -0.0415 0.02785" rpy="0.0 ${pi/2} ${pi/2}"/>
+            <geometry>
+                <mesh filename="package://hexapod_description/meshes/gripper_hand.stl" scale="0.001 0.001 0.001"/>
+            </geometry>
+            <material name="">
+                <color rgba="1.0 1.0 1.0 1.0"/>
+            </material>
+        </collision>
+        <inertial>
+            <origin xyz="0.0 0.0 0.0" rpy="0.0 0.0 0.0" />
+            <mass value="0.00001"/>
+            <inertia
+                ixx="1.0" ixy="0.0"  ixz="0.0"
+                iyy="1.0" iyz="0.0"
+                izz="1.0" />
+        </inertial>
+    </link>
+    <gazebo reference="pan_link">
+        <material>Gazebo/DarkGrey</material>
+    </gazebo>
     <!-- Leg macro -->
     <xacro:macro name="leg" params="side position x y angle axis">
@@ -124,5 +173,6 @@
         <!-- femur -->
         <joint name="femur_joint_${side}${position}" type="revolute">
-            <origin xyz="${coxa_length} 0.0 0.0" rpy="${pi/2} ${pi/2} 0.0"/>
+            <!-- <origin xyz="${coxa_length} 0.0 0.0" rpy="${pi/2} ${pi/2} 0.0"/> -->
+            <origin xyz="${coxa_length} 0.0 0.0" rpy="${pi/2} ${pi/3} 0.0"/>
             <parent link="coxa_${side}${position}"/>
             <child link="femur_${side}${position}"/>
@@ -173,5 +223,6 @@
         <!-- tibia -->
         <joint name="tibia_joint_${side}${position}" type="revolute">
-            <origin xyz="0.0 ${femur_length} 0.0" rpy="0.0 0.0 0.0"/>
+            <!-- <origin xyz="0.0 ${femur_length} 0.0" rpy="0.0 0.0 0.0"/> -->
+            <origin xyz="0.0 ${femur_length} 0.0" rpy="0.0 0.0 ${pi/6}"/>
             <parent link="femur_${side}${position}"/>
             <child link="tibia_${side}${position}"/>
@@ -191,5 +242,6 @@
         <link name="tibia_${side}${position}">
             <visual>
-                <origin xyz="0.02285 -0.01325 -0.0205" rpy="0.0 0.0 ${pi/2}"/>
+                <!-- <origin xyz="0.02285 -0.01325 -0.0205" rpy="0.0 0.0 ${pi/2}"/> -->
+                <origin xyz="-0.01285 -0.0237 -0.0205" rpy="0.0 0.0 0.0"/>
                 <geometry>
                     <mesh filename="package://hexapod_description/meshes/tibia.stl" scale="0.001 0.001 0.001"/>
@@ -219,4 +271,30 @@
         <gazebo reference="tibia_${side}${position}">
             <material>Gazebo/DarkGrey</material>
+        </gazebo>
+        <!-- foot -->
+        <joint name="foot_joint_${side}${position}" type="fixed">
+            <!-- <origin xyz="0.0 ${tibia_length} 0.0" rpy="0.0 0.0 0.0" /> -->
+            <origin xyz="${tibia_length} 0.0 0.0" rpy="0.0 0.0 0.0" />
+            <parent link="tibia_${side}${position}" />
+            <child link="foot_${side}${position}" />
+        </joint>
+        <link name="foot_${side}${position}">
+            <inertial>
+                <origin xyz="0.0 0.0 0.0" rpy="0.0 0.0 0.0" />
+                <mass value="0.00001"/>
+                <inertia
+                    ixx="1.0" ixy="0.0"  ixz="0.0"
+                    iyy="1.0" iyz="0.0"
+                    izz="1.0" />
+            </inertial>
+        </link>
+        <gazebo>
+            <plugin name="f3d_controller" filename="libgazebo_ros_f3d.so">
+                <alwaysOn>true</alwaysOn>
+                <updateRate>50</updateRate>
+                <bodyName>foot_${side}${position}</bodyName>
+                <topicName>${side}${position}_ground_feedback</topicName>
+                <frameName>foot_${side}${position}</frameName>
+            </plugin>
         </gazebo>
     </xacro:macro>

Commit message: ...

File: hexapod_description/urdf/ancabot.xacro (robot description, xacro)
@@ -8,5 +8,5 @@
     <xacro:property     name="femur_length"     value="0.042"/>
     <xacro:property     name="tibia_length"     value="0.0665"/>
-    <xacro:property     name="ground_offset"    value="0.065" />
+    <xacro:property     name="ground_offset"    value="0.095" />
     <gazebo>
         <plugin name="gazebo_ros_control" filename="libgazebo_ros_control.so">

Commit message: ...

File: hexapod_description/urdf/ancabot.xacro (robot description, xacro)
@@ -54,6 +54,6 @@
     <xacro:property name="joint_lower_limit" value="-${2.0}"/>
     <xacro:property name="joint_upper_limit" value="${2.0}"/>
-    <xacro:property name="joint_effort" value="6.0"/>
-    <xacro:property name="joint_velocity" value="0.524"/>
+    <xacro:property name="joint_effort" value="20.0"/>
+    <xacro:property name="joint_velocity" value="0.75"/>
     <!-- Head properties -->
     <joint name="pan_joint" type="revolute">
@@ -173,5 +173,4 @@
         <!-- femur -->
         <joint name="femur_joint_${side}${position}" type="revolute">
-            <!-- <origin xyz="${coxa_length} 0.0 0.0" rpy="${pi/2} ${pi/2} 0.0"/> -->
             <origin xyz="${coxa_length} 0.0 0.0" rpy="${pi/2} ${pi/3} 0.0"/>
             <parent link="coxa_${side}${position}"/>
@@ -242,5 +241,4 @@
         <link name="tibia_${side}${position}">
             <visual>
-                <!-- <origin xyz="0.02285 -0.01325 -0.0205" rpy="0.0 0.0 ${pi/2}"/> -->
                 <origin xyz="-0.01285 -0.0237 -0.0205" rpy="0.0 0.0 0.0"/>
                 <geometry>
@@ -252,5 +250,5 @@
             </visual>
             <collision>
-                <origin xyz="0.02285 -0.01325 -0.0205" rpy="0.0 0.0 ${pi/2}"/>
+                <origin xyz="-0.01285 -0.0237 -0.0205" rpy="0.0 0.0 0.0"/>
                 <geometry>
                     <mesh filename="package://hexapod_description/meshes/tibia.stl" scale="0.001 0.001 0.001"/>
