Commit message: update

File: hexapod_description/urdf/ancabot_model.xacro (robot description, xacro)
@@ -1,4 +1,31 @@
 <?xml version="1.0" encoding="UTF-8" ?>
 <robot xmlns:xacro="http://ros.org/wiki/xacro" name="Ancabot">
+    <xacro:macro name="inertial_sphere" params="mass radius *origin">
+        <inertial>
+            <xacro:insert_block name="origin"/>
+            <mass value="${mass}" />
+            <inertia ixx="${(2/5) * mass * (radius*radius)}" ixy="0.0" ixz="0.0"
+                    iyy="${(2/5) * mass * (radius*radius)}" iyz="0.0"
+                    izz="${(2/5) * mass * (radius*radius)}" />
+        </inertial>
+    </xacro:macro>
+    <xacro:macro name="inertial_box" params="mass x y z *origin">
+        <inertial>
+            <xacro:insert_block name="origin"/>
+            <mass value="${mass}" />
+            <inertia ixx="${(1/12) * mass * (y*y+z*z)}" ixy="0.0" ixz="0.0"
+                    iyy="${(1/12) * mass * (x*x+z*z)}" iyz="0.0"
+                    izz="${(1/12) * mass * (x*x+y*y)}" />
+        </inertial>
+    </xacro:macro>
+    <xacro:macro name="inertial_cylinder" params="mass length radius *origin">
+        <inertial>
+            <xacro:insert_block name="origin"/>
+            <mass value="${mass}" />
+            <inertia ixx="${(1/12) * mass * (3*radius*radius + length*length)}" ixy="0.0" ixz="0.0"
+                    iyy="${(1/12) * mass * (3*radius*radius + length*length)}" iyz="0.0"
+                    izz="${(1/2) * mass * (radius*radius)}" />
+        </inertial>
+    </xacro:macro>
     <!-- parameters -->
     <xacro:property     name="body_length"      value="0.2425"/>
@@ -34,12 +61,7 @@
             </material>
         </collision>
-        <inertial>
-            <origin xyz="0.0 0.0 0.0" rpy="0.0 0.0 0.0" />
-            <mass value="0.00001"/>
-            <inertia
-                ixx="1.0" ixy="0.0"  ixz="0.0"
-                iyy="1.0" iyz="0.0"
-                izz="1.0" />
-        </inertial>
+        <xacro:inertial_box mass="1.031" x="${body_width}" y="${body_length}" z="${body_height}">
+            <origin xyz="0.0 0.05 0.0" rpy="0.0 0.0 0.0"/>
+        </xacro:inertial_box>
     </link>
     <gazebo reference="body_link">
@@ -92,12 +114,7 @@
             </material>
         </collision>
-        <inertial>
-            <origin xyz="0.0 0.0 0.0" rpy="0.0 0.0 0.0" />
-            <mass value="0.00001"/>
-            <inertia
-                ixx="1.0" ixy="0.0"  ixz="0.0"
-                iyy="1.0" iyz="0.0"
-                izz="1.0" />
-        </inertial>
+        <xacro:inertial_cylinder mass="0.0125" length="0.055" radius="0.02">
+            <origin xyz="0.02 0.02 0.0" rpy="0.0 ${pi/2} 0.0"/>
+        </xacro:inertial_cylinder>
     </link>
     <gazebo reference="pan_link">
@@ -113,12 +130,16 @@
         </joint>
         <link name="leg_center_${side}${position}">
-            <inertial>
-                <origin xyz="0.0 0.0 0.0" rpy="0.0 0.0 0.0" />
-                <mass value="0.00001"/>
-                <inertia
-                    ixx="1.0" ixy="0.0"  ixz="0.0"
-                    iyy="1.0" iyz="0.0"
-                    izz="1.0" />
-            </inertial>
+        <collision>
+                <origin xyz="0.0 0.0 0.0" rpy="0.0 0.0 0.0"/>
+                <geometry>
+                    <cylinder length="0.02" radius="0.02"/>
+                </geometry>
+                <material name="">
+                    <color rgba="1.0 1.0 1.0 1.0"/>
+                </material>
+            </collision>
+            <xacro:inertial_cylinder mass="0.02" length="0.02" radius="0.02">
+                <origin xyz="0.0 0.0 0.0" rpy="0.0 0.0 0.0"/>
+            </xacro:inertial_cylinder>
         </link>
         <!-- coxa -->
@@ -159,12 +180,7 @@
                 </material>
             </collision>
-            <inertial>
-                <origin xyz="0.0 0.0 0.0" rpy="0.0 0.0 0.0" />
-                <mass value="0.00001"/>
-                <inertia
-                    ixx="1.0" ixy="0.0"  ixz="0.0"
-                    iyy="1.0" iyz="0.0"
-                    izz="1.0" />
-            </inertial>
+            <xacro:inertial_cylinder mass="0.02" length="0.0475" radius="0.02">
+                <origin xyz="0.02 0.02 0.0" rpy="0.0 ${pi/2} 0.0"/>
+            </xacro:inertial_cylinder>
         </link>
         <gazebo reference="coxa_${side}${position}">
@@ -208,12 +224,7 @@
                 </material>
             </collision>
-            <inertial>
-                <origin xyz="0.0 0.0 0.0" rpy="0.0 0.0 0.0" />
-                <mass value="0.00001"/>
-                <inertia
-                    ixx="1.0" ixy="0.0"  ixz="0.0"
-                    iyy="1.0" iyz="0.0"
-                    izz="1.0" />
-            </inertial>
+            <xacro:inertial_cylinder mass="0.184" length="0.0475" radius="0.02">
+                <origin xyz="0.0 0.02375 0.0" rpy="${pi/2} 0.0 0.0"/>
+            </xacro:inertial_cylinder>
         </link>
         <gazebo reference="femur_${side}${position}">
@@ -258,12 +269,7 @@
                 </material>
             </collision>
-            <inertial>
-                <origin xyz="0.0 0.0 0.0" rpy="0.0 0.0 0.0" />
-                <mass value="0.00001"/>
-                <inertia
-                    ixx="1.0" ixy="0.0"  ixz="0.0"
-                    iyy="1.0" iyz="0.0"
-                    izz="1.0" />
-            </inertial>
+            <xacro:inertial_cylinder mass="0.184" length="0.0775" radius="0.02">
+                <origin xyz="0.02375 0.0 0.0" rpy="0.0 ${pi/2} 0.0"/>
+            </xacro:inertial_cylinder>
         </link>
         <gazebo reference="tibia_${side}${position}">
@@ -271,5 +277,5 @@
         </gazebo>
         <!-- foot -->
-        <joint name="foot_joint_${side}${position}" type="fixed">
+        <!-- <joint name="foot_joint_${side}${position}" type="fixed">
             <origin xyz="${tibia_length} 0.0 0.0" rpy="0.0 0.0 0.0" />
             <parent link="tibia_${side}${position}" />
@@ -277,12 +283,16 @@
         </joint>
         <link name="foot_${side}${position}">
-            <inertial>
-                <origin xyz="0.0 0.0 0.0" rpy="0.0 0.0 0.0" />
-                <mass value="0.00001"/>
-                <inertia
-                    ixx="1.0" ixy="0.0"  ixz="0.0"
-                    iyy="1.0" iyz="0.0"
-                    izz="1.0" />
-            </inertial>
+            <collision>
+                <origin xyz="0.0 0.0 0.0" rpy="0.0 0.0 0.0"/>
+                <geometry>
+                    <sphere radius="0.02"/>
+                </geometry>
+                <material name="">
+                    <color rgba="1.0 1.0 1.0 1.0"/>
+                </material>
+            </collision>
+            <xacro:inertial_sphere mass="0.02" radius="0.02">
+                <origin xyz="0.0 0.0 0.0" rpy="0.0 0.0 0.0"/>
+            </xacro:inertial_sphere>
         </link>
         <gazebo>
@@ -294,5 +304,5 @@
                 <frameName>foot_${side}${position}</frameName>
             </plugin>
-        </gazebo>
+        </gazebo> -->
     </xacro:macro>
     <!-- Build robot model -->

Commit message: ...

File: hexapod_description/urdf/ancabot_model.xacro (robot description, xacro)
@@ -115,5 +115,5 @@
         </collision>
         <xacro:inertial_cylinder mass="0.0125" length="0.055" radius="0.02">
-            <origin xyz="0.02 0.02 0.0" rpy="0.0 ${pi/2} 0.0"/>
+            <origin xyz="0.05 0.05 0.0" rpy="0.0 ${pi/2} 0.0"/>
         </xacro:inertial_cylinder>
     </link>
